Commit message: changed 2 wheels to 4 wheels.

File: description/robot_core.xacro (robot description, xacro)
@@ -21,22 +21,22 @@
         <parent link="base_link"/>
         <child link="chassis"/>
-        <origin xyz="-0.1 0 0"/>
+        <origin xyz="-0.25 0 0"/>
     </joint>
     <link name="chassis">
         <visual>
-            <origin xyz="0.15 0 0.075"/>
+            <origin xyz="0.25 0 0.075"/>
             <geometry>
-                <box size="0.3 0.3 0.15"/>
+                <box size="0.5 0.3 0.15"/>
             </geometry>
             <material name="white"/>
         </visual>
         <collision>
-            <origin xyz="0.15 0 0.075"/>
+            <origin xyz="0.25 0 0.075"/>
             <geometry>
-                <box size="0.3 0.3 0.15"/>
+                <box size="0.5 0.3 0.15"/>
             </geometry>
         </collision>
-        <xacro:inertial_box mass="0.5" x="0.3" y="0.3" z="0.15">
-            <origin xyz="0.15 0 0.075" rpy="0 0 0"/>
+        <xacro:inertial_box mass="0.5" x="0.5" y="0.3" z="0.15">
+            <origin xyz="0.3 0 0.075" rpy="0 0 0"/>
         </xacro:inertial_box>
     </link>
@@ -45,8 +45,54 @@
         <parent link="base_link"/>
         <child link="left_wheel"/>
-        <origin xyz="0 0.175 0" rpy="-${pi/2} 0 0" />
+        <origin xyz="-0.20 0.175 0" rpy="-${pi/2} 0 0" />
         <axis xyz="0 0 1"/>
     </joint>
     <link name="left_wheel">
+        <visual>
+            <geometry>
+                <cylinder radius="0.05" length="0.04"/>
+            </geometry>
+            <material name="blue"/>
+        </visual>
+        <collision>
+            <geometry>
+                <cylinder radius="0.05" length="0.04"/>
+            </geometry>
+        </collision>
+        <xacro:inertial_cylinder mass="0.1" length="0.04" radius="0.05">
+            <origin xyz="0 0 0" rpy="0 0 0"/>
+        </xacro:inertial_cylinder>
+    </link>
+    <!-- FRONT LEFT WHEEL LINK -->
+    <joint name="front_left_wheel_joint" type="continuous">
+        <parent link="base_link"/>
+        <child link="front_left_wheel"/>
+        <origin xyz="0.20 0.175 0" rpy="-${pi/2} 0 0" />
+        <axis xyz="0 0 1"/>
+    </joint>
+    <link name="front_left_wheel">
+        <visual>
+            <geometry>
+                <cylinder radius="0.05" length="0.04"/>
+            </geometry>
+            <material name="blue"/>
+        </visual>
+        <collision>
+            <geometry>
+                <cylinder radius="0.05" length="0.04"/>
+            </geometry>
+        </collision>
+        <xacro:inertial_cylinder mass="0.1" length="0.04" radius="0.05">
+            <origin xyz="0 0 0" rpy="0 0 0"/>
+        </xacro:inertial_cylinder>
+    </link>
+    <!-- FRONT RIGHT WHEEL LINK -->
+    <joint name="front_right_wheel_joint" type="continuous">
+        <parent link="base_link"/>
+        <child link="front_right_wheel"/>
+        <origin xyz="0.20 -0.175 0" rpy="${pi/2} 0 0" />
+        <axis xyz="0 0 -1"/>
+    </joint>
+    <link name="front_right_wheel">
         <visual>
             <geometry>
@@ -68,5 +114,5 @@
         <parent link="base_link"/>
         <child link="right_wheel"/>
-        <origin xyz="0 -0.175 0" rpy="${pi/2} 0 0" />
+        <origin xyz="-0.20 -0.175 0" rpy="${pi/2} 0 0" />
         <axis xyz="0 0 -1"/>
     </joint>
@@ -87,25 +133,3 @@
         </xacro:inertial_cylinder>
     </link>
-    <!-- CASTER WHEEL LINK -->
-    <joint name="caster_wheel_joint" type="fixed">
-        <parent link="chassis"/>
-        <child link="caster_wheel"/>
-        <origin xyz="0.24 0 0"/>
-    </joint>
-    <link name="caster_wheel">
-        <visual>
-            <geometry>
-                <sphere radius="0.05"/>
-            </geometry>
-            <material name="black"/>
-        </visual>
-        <collision>
-            <geometry>
-                <sphere radius="0.05"/>
-            </geometry>
-        </collision>
-        <xacro:inertial_sphere mass="0.1" radius="0.05">
-            <origin xyz="0 0 0" rpy="0 0 0"/>
-        </xacro:inertial_sphere>
-    </link>
 </robot>

Commit message: lidar integration

File: description/robot_core.xacro (robot description, xacro)
@@ -65,5 +65,5 @@
     </link>
     <!-- FRONT LEFT WHEEL LINK -->
-    <joint name="front_left_wheel_joint" type="fixed">
+    <joint name="front_left_wheel_joint" type="continuous">
         <parent link="base_link"/>
         <child link="front_left_wheel"/>
@@ -88,5 +88,5 @@
     </link>
     <!-- FRONT RIGHT WHEEL LINK -->
-    <joint name="front_right_wheel_joint" type="fixed">
+    <joint name="front_right_wheel_joint" type="continuous">
         <parent link="base_link"/>
         <child link="front_right_wheel"/>

Commit message: base_footprint added

File: description/robot_core.xacro (robot description, xacro)
@@ -16,4 +16,11 @@
     <!-- BASE LINK -->
     <link name="base_link">
+    </link>
+    <joint name="base_footprint_joint" type="fixed">
+        <parent link="base_link"/>
+        <child link="base_footprint"/>
+        <origin xyz="0 0 0" rpy="0 0 0"/>
+    </joint>
+    <link name="base_footprint">
     </link>
     <!-- CHASSIS LINK -->

Commit message: scripts added

File: description/robot_core.xacro (robot description, xacro)
@@ -66,12 +66,4 @@
                 <cylinder radius="0.05" length="0.04"/>
             </geometry>
-            <surface>
-                <friction>
-                    <ode>
-                        <mu>1.0</mu>          <!-- Coefficient of friction -->
-                        <mu2>0.5</mu2>        <!-- Orthogonal friction -->
-                    </ode>
-                </friction>
-            </surface>
         </collision>
         <xacro:inertial_cylinder mass="0.1" length="0.04" radius="0.05">
@@ -97,12 +89,4 @@
                 <cylinder radius="0.05" length="0.04"/>
             </geometry>
-            <surface>
-                <friction>
-                    <ode>
-                        <mu>1.0</mu>          <!-- Coefficient of friction -->
-                        <mu2>0.5</mu2>        <!-- Orthogonal friction -->
-                    </ode>
-                </friction>
-            </surface>
         </collision>
         <xacro:inertial_cylinder mass="0.1" length="0.04" radius="0.05">
@@ -128,12 +112,4 @@
                 <cylinder radius="0.05" length="0.04"/>
             </geometry>
-            <surface>
-                <friction>
-                    <ode>
-                        <mu>1.0</mu>          <!-- Coefficient of friction -->
-                        <mu2>0.5</mu2>        <!-- Orthogonal friction -->
-                    </ode>
-                </friction>
-            </surface>
         </collision>
         <xacro:inertial_cylinder mass="0.1" length="0.04" radius="0.05">
@@ -159,12 +135,4 @@
                 <cylinder radius="0.05" length="0.04"/>
             </geometry>
-            <surface>
-                <friction>
-                    <ode>
-                        <mu>1.0</mu>          <!-- Coefficient of friction -->
-                        <mu2>0.5</mu2>        <!-- Orthogonal friction -->
-                    </ode>
-                </friction>
-            </surface>
         </collision>
         <xacro:inertial_cylinder mass="0.1" length="0.04" radius="0.05">
@@ -172,3 +140,13 @@
         </xacro:inertial_cylinder>
     </link>
+	<gazebo reference="front_right_wheel">
+ 	       <material>Gazebo/Black</material>
+ 	       <mu1 value="0.001"/>
+ 	       <mu2 value="0.001"/>
+ 	</gazebo>
+ 	<gazebo reference="front_left_wheel">
+ 	       <material>Gazebo/Black</material>
+ 	       <mu1 value="0.001"/>
+ 	       <mu2 value="0.001"/>
+ 	</gazebo>
 </robot>
